File: hardware/the-card.kicad_sch (KiCad schematic)
At the start: 0 parts

Commit message: feat(hardware): generate the-card.kicad_sch directly from circuit.py
gen_schematic.py builds the KiCad schematic in code (no GUI, no skidl auto-layout):
- embeds symbol defs from our .kicad_sym libraries
- places all 53 parts on a 1.27mm grid
- net-labels every pin (skidl pin coords; Y negated vs KiCad)
- marks intentionally-unused pins with no_connect
- sets embedded pins to passive type (easyeda mistypes them) for clean ERC

Result: the-card.kicad_sch loads in KiCad 10, ERC = 0 errors / 18 expected
warnings (single-pin pass-through nets: NFC antenna, e-ink booster, motor).
Parts:
- added C_bat, C_imu2, C_mcu2, C_vbus: 10uF, Capacitor_SMD:C_0603_1608Metric, symbol passives:CL10A106KP8NNNC
- added C_btn1, C_btn2, C_btn3, C_btn4, C_dprot, C_fg, C_imu1, C_led, C_mcu1, C_nfc, C_sht, C_vb: 100nF, Capacitor_SMD:C_0402_1005Metric, symbol passives:CL05B104KO5NNNC
- added C_en, C_epdvdd, C_ldoi, C_ldoo: 1uF, Capacitor_SMD:C_0603_1608Metric, symbol passives:CL10A106KP8NNNC
- added D1: WS2812B-MINI, symbol the-card:WS2812B-MINI
- added J1: TYPE-C-31-M-12, symbol the-card:TYPE-C-31-M-12
- added J2: FPC 0.5-24P LTH2.0, symbol the-card:FPC0.5-24PLTH2.0
- added Q1, Q2: SI2301CDS-T1-GE3, symbol the-card:SI2301CDS-T1-GE3
- added R_cc1, R_cc2: 5.1k, Resistor_SMD:R_0402_1005Metric, symbol passives:0402WGF1002TCE
- added R_chrg, R_en, R_io0, R_q1g, R_q2g: 10k, Resistor_SMD:R_0402_1005Metric, symbol passives:0402WGF1002TCE
- added R_dvcc: 470, Resistor_SMD:R_0402_1005Metric, symbol passives:0402WGF1002TCE
- added R_dvm: 2k, Resistor_SMD:R_0402_1005Metric, symbol passives:0402WGF1002TCE
- added R_prog: 1.2k, Resistor_SMD:R_0402_1005Metric, symbol passives:0402WGF1002TCE
- added R_scl, R_sda: 4.7k, Resistor_SMD:R_0402_1005Metric, symbol passives:0402WGF1002TCE
- added R_vbh: 1M, Resistor_SMD:R_0402_1005Metric, symbol passives:0402WGF1002TCE
- added R_vbl: 300k, Resistor_SMD:R_0402_1005Metric, symbol passives:0402WGF1002TCE
- added SW1, SW2, SW3, SW4: TS-1187A-B-A-B, symbol the-card:TS-1187A-B-A-B
- added U1: ESP32-S3-WROOM-1-N8R2, symbol the-card:ESP32-S3-WROOM-1
- added U10: USBLC6-2SC6, symbol the-card:USBLC6-2SC6
- added U2: ST25DV04KC-IE8S3, symbol the-card:ST25DV04KC-IE8S3
- added U3: LSM6DSOTR, symbol the-card:LSM6DSOTR
- added U4: SHT40-BD1B-R2, symbol the-card:SHT40-BD1B-R2
- added U5: MAX17048G+T10, symbol the-card:MAX17048G+T10
- added U6: TP4056_C382139, symbol the-card:TP4056_C382139
- added U7: DW01A_C18164398, symbol the-card:DW01A_C18164398
- added U8: FS8205A, symbol the-card:FS8205A
- added U9: ME6211C33M5G-N, symbol the-card:ME6211C33M5G-N
Connections:
- new net +3V3: C_ldoo.1, C_mcu1.1, C_mcu2.1, C_nfc.1, Q1.2 (S), Q2.2 (S), R_chrg.1, R_en.1, R_io0.1, R_q1g.1, R_q2g.1, R_scl.1, R_sda.1, U1.2 (3V3), U2.8 (VCC), U9.5 (VOUT)
- new net +BAT: C_bat.1, C_fg.1, C_ldoi.1, R_dvcc.1, R_vbh.1, U5.2 (CELL), U5.3 (VDD), U6.5 (BAT), U9.1 (VIN), U9.3 (CE)
- new net AUX_3V3: C_imu1.1, C_imu2.1, C_led.1, C_sht.1, D1.1 (VDD), Q1.3 (D), U3.12 (CS), U3.5 (VDDIO), U3.8 (VDD), U4.3 (VDD)
- new net BAT_NEG: C_dprot.2, U7.6 (VSS), U8.2 (S1), U8.3 (S1)
- new net BTN_DOWN: C_btn2.1, SW2.1 (A), U1.5 (IO5)
- new net BTN_MENU: C_btn4.1, SW4.1 (A), U1.7 (IO7)
- new net BTN_SEL: C_btn3.1, SW3.1 (A), U1.6 (IO6)
- new net BTN_UP: C_btn1.1, SW1.1 (A), U1.4 (IO4)
- new net EPD_BUSY: J2.9, U1.19 (IO11)
- new net EPD_CS: J2.12, U1.20 (IO12)
- new net EPD_DC: J2.11, U1.21 (IO13)
- new net EPD_GDR: J2.2
- new net EPD_NC1: J2.1
- new net EPD_NC4: J2.4
- new net EPD_PWR_EN: Q2.1 (G), R_q2g.2, U1.9 (IO16)
- new net EPD_RESE: J2.3
- new net EPD_RST: J2.10, U1.22 (IO14)
- new net EPD_SCLK: J2.13, U1.18 (IO10)
- new net EPD_SDA: J2.14, U1.17 (IO9)
- new net EPD_TSCL: J2.6
- new net EPD_TSDA: J2.7
- new net EPD_VCOM: J2.24
- new net EPD_VDD: J2.15, J2.16, Q2.3 (D)
- new net EPD_VGH: J2.21
- new net EPD_VGL: J2.23
- new net EPD_VPP: J2.19
- new net EPD_VSH1: J2.20
- new net EPD_VSH2: J2.5
- new net EPD_VSL: J2.22
- new net FET_DRAIN: U8.1 (D12), U8.8 (D12)
- new net GND: C_bat.2, C_btn1.2, C_btn2.2, C_btn3.2, C_btn4.2, C_en.2, C_epdvdd.2, C_fg.2, C_imu1.2, C_imu2.2, C_ldoi.2, C_ldoo.2, C_led.2, C_mcu1.2, C_mcu2.2, C_nfc.2, C_sht.2, C_vb.2, C_vbus.2, D1.3 (VSS), J1.1 (EH), J1.2 (EH), J1.3 (EH), J1.4 (EH), J1.A1B12 (GND), J1.B1A12 (GND), J2.17, J2.25, J2.26, J2.8, R_cc1.2, R_cc2.2, R_dvm.1, R_prog.2, R_vbl.2, SW1.3 (C), SW2.3 (C), SW3.3 (C), SW4.3 (C), U1.1 (GND), U1.40 (GND), U1.41 (GND), U10.2, U2.4 (VSS), U3.1 (SDO/SA0), U3.6 (GND), U3.7 (GND), U4.4 (VSS), U4.5 (EP), U5.1 (CTG), U5.4 (GND), U5.6 (QSTRT), U5.9 (EP), U6.1 (TEMP), U6.3 (GND), U6.9 (EP), U8.6 (S2), U8.7 (S2), U9.2 (VSS)
- new net I2C_SCL: R_scl.2, U1.12 (IO8), U2.6 (SCL), U3.13 (SCL), U4.2 (SCL), U5.7 (SCL)
- new net I2C_SDA: R_sda.2, U1.11 (IO18), U2.5 (SDA), U3.14 (SDA), U4.1 (SDA), U5.8 (SDA)
- new net IMU_INT: U1.38 (IO2), U3.4 (INT1)
- new net LED_DIN: D1.4 (DIN), U1.25 (IO48)
- new net MOTOR_PWM: U1.23 (IO21)
- new net N$1: C_en.1, R_en.2, U1.3 (EN)
- new net N$10: C_dprot.1, R_dvcc.2, U7.5 (VDD)
- new net N$11: R_dvm.2, U7.2 (VM)
- new net N$12: U7.3 (COUT), U8.4 (G1)
- new net N$13: U7.1 (DOUT), U8.5 (G2)
- new net N$14: C_epdvdd.1, J2.18
- new net N$2: R_io0.2, U1.27 (IO0)
- new net N$3: C_vb.1, R_vbh.2, R_vbl.1, U1.39 (IO1)
- new net N$4: J1.A5 (CC1), R_cc1.1
- new net N$5: J1.B5 (CC2), R_cc2.1
- new net N$6: J1.A7 (DN1), J1.B7 (DN2), U10.1
- new net N$7: J1.A6 (DP1), J1.B6 (DP2), U10.3
- new net N$8: R_prog.1, U6.2 (PROG)
- new net N$9: R_chrg.2, U6.7 (~{CHRG})
- new net NFC_ANT_A: U2.2 (AC0)
- new net NFC_ANT_B: U2.3 (AC1)
- new net NFC_EH: U2.1 (V_EH)
- new net NFC_IRQ: U1.15 (IO3), U2.7 (GPO)
- new net PWR_AUX: Q1.1 (G), R_q1g.2, U1.24 (IO47)
- new net USB_DM: U1.13 (IO19), U10.6
- new net USB_DP: U1.14 (IO20), U10.4
- new net VBUS: C_vbus.1, J1.A4B9 (VBUS), J1.B4A9 (VBUS), U10.5, U6.4 (VCC), U6.8 (CE)
- new net ~CHRG: U1.8 (IO15)
- no-connect marks 0 -> 33

Commit message: feat(hardware): v2 schematic gen — subsystem grouping + power symbols
gen_schematic.py now:
- groups parts into 5 labelled bands (POWER/MCU/DISPLAY/SENSORS/UI)
- uses real KiCad power symbols (GND/+3V3/+BAT/VBUS/AUX_3V3/EPD_VDD) from the
  installed power.kicad_sym, with one PWR_FLAG per rail (power_out pin)
- collision-aware placement (no cross-net pin-endpoint coincidences)
- snaps to the 1.27 mm grid

ERC: 0 errors (41 expected warnings: custom power symbols not in stock lib +
single-pin pass-through nets). Renders to PDF.
Other:
- note added: "E-INK DISPLAY"
- note added: "MCU — ESP32-S3"
- note added: "POWER SUPPLY & CHARGING"
- note added: "SENSORS & NFC (I2C)"
- note added: "USER INTERFACE"

Commit message: feat(hardware): v3 schematic — hand-crafted placement + local wires
Replaces the uniform grid with a hand-designed layout: power chain top-left,
MCU centre, I²C sensors on the left, e-ink/LED below, buttons at the bottom,
decoupling caps against their ICs. Keeps KiCad power symbols + PWR_FLAG rails,
net labels for MCU-fanout signals (correct for an MCU board), and direct wires
for the few close 2-pin signal nets. ERC: 0 errors.
Connections:
- net FET_DRAIN: no longer names the net of U8.1 (D12), U8.8 (D12)
- net N$14: no longer names the net of C_epdvdd.1, J2.18
Other:
- note removed: "E-INK DISPLAY"
- note removed: "MCU — ESP32-S3"
- note removed: "POWER SUPPLY & CHARGING"
- note removed: "SENSORS & NFC (I2C)"
- note removed: "USER INTERFACE"

Commit message: feat(hardware): v4 schematic — pin-cluster placement, 13 direct wires
Peripherals placed on the MCU side where their signal pins are:
  SPI bus (6 wires) below · buttons (4 wires) + USB (2) + LED (1) on left/bottom.
Point-to-point nets become short L-wires; shared buses (I2C) stay labels.
ERC: 0 errors (44 expected warnings).
Connections:
- net EPD_BUSY is gone; now on net EPD_GDR: J2.9, U1.19 (IO11)
- net EPD_CS is gone; now on net EPD_GDR: J2.12, U1.20 (IO12)
- net EPD_DC is gone; now on net EPD_GDR: J2.11, U1.21 (IO13)
- net EPD_NC1 is gone; now on net EPD_GDR: J2.1
- net EPD_NC4 is gone; now on net EPD_GDR: J2.4
- net EPD_RESE is gone; now on net EPD_GDR: J2.3
- net EPD_RST is gone; now on net EPD_GDR: J2.10, U1.22 (IO14)
- net EPD_SCLK is gone; now on net EPD_GDR: J2.13, U1.18 (IO10)
- net EPD_SDA is gone; now on net EPD_GDR: J2.14, U1.17 (IO9)
- net EPD_TSCL is gone; now on net EPD_GDR: J2.6
- net EPD_TSDA is gone; now on net EPD_GDR: J2.7
- net EPD_VSH2 is gone; now on net EPD_GDR: J2.5
- net N$13 is gone; now on net BAT_NEG: U7.1 (DOUT), U8.5 (G2)
- net N$4 is gone; now on net AUX_3V3: J1.A5 (CC1), R_cc1.1
- net N$5 is gone; now on net AUX_3V3: J1.B5 (CC2), R_cc2.1
- net NFC_IRQ is gone; now on net EPD_GDR: U1.15 (IO3), U2.7 (GPO)
- net PWR_AUX is gone; now on net EPD_GDR: Q1.1 (G), R_q1g.2, U1.24 (IO47)
- net AUX_3V3: now also C_epdvdd.1, J2.18
- net LED_DIN: no longer names the net of D1.4 (DIN), U1.25 (IO48)
- net N$12: no longer names the net of U7.3 (COUT), U8.4 (G1)
- net N$2: no longer names the net of R_io0.2, U1.27 (IO0)
- net USB_DM: no longer names the net of U1.13 (IO19), U10.6

Commit message: fix(hardware): v3.1 — hand-crafted layout + 13 wires (v3 placement, WIRE_MAX=120)
Reverts to v3's hand-crafted placement (signal-flow, not pin-cluster auto-placement)
but extends the 2-pin wire threshold to 120 mm, capturing 13 direct L-wires
(SPI bus, buttons, USB, LED, etc.) while keeping the proven layout. ERC: 0 errors.
Connections:
- net N$9 is gone; now on an unnamed net: R_chrg.2, U6.7 (~{CHRG})
- net AUX_3V3: no longer C_epdvdd.1, J1.A5 (CC1), J1.B5 (CC2), J2.18, R_cc1.1, R_cc2.1
- net EPD_GDR: no longer Q1.1 (G), R_q1g.2, U1.24 (IO47)
- net USB_DM: now reaches U1.13 (IO19), U10.6
- net LED_DIN: now reaches D1.4 (DIN), U1.25 (IO48)
- net N$8: no longer names the net of R_prog.1, U6.2 (PROG)
- new net: C_epdvdd.1, J2.18
- new net N$4: J1.A5 (CC1), R_cc1.1
- new net N$5: J1.B5 (CC2), R_cc2.1
- new net PWR_AUX: Q1.1 (G), R_q1g.2, U1.24 (IO47)

Commit message: fix(hardware): improved placement — USB near MCU, sensors hug I2C, caps on ICs
- USB-C + ESD moved from power area to MCU left side (near USB_DM/DP pins)
- Sensors shifted right to ~x310 (close to MCU I2C pins at ~x398)
- Buttons raised from y=320 to y=385 (closer to BTN pin row)
- Decoupling caps placed directly above their ICs (C_mcu1/2 at y=152, U1 at y=220)
- Collision avoidance restored (prevents PWR_FLAG pin_to_pin)
ERC: 0 errors, 13 wires.
Connections:
- net EPD_GDR renamed EPD_DC
- net LED_DIN: no longer names the net of D1.4 (DIN), U1.25 (IO48)

Commit message: feat(hardware): add single-page schematic layout
Parts:
- D1: footprint (none) -> the-card:LED-SMD_4P-L3.5-W3.5-TL_WS2812B
- J1: footprint (none) -> the-card:USB-C_SMD-TYPE-C-31-M-12_1
- J2: footprint (none) -> the-card:FPC-SMD_FPC-0.5-24P-LTH2.0
- Q1, Q2: footprint (none) -> the-card:SOT-23-3_L3.0-W1.7-P0.95-LS2.9-BR
- SW1, SW2, SW3, SW4: footprint (none) -> the-card:SW-SMD_4P-L5.1-W5.1-P3.70-LS6.5-TL_H1.5
- U1: footprint (none) -> the-card:WIRELM-SMD_ESP32-S3-WROOM-1
- U10: footprint (none) -> the-card:SOT-23-6_L2.9-W1.6-P0.95-LS2.8-BL
- U2: footprint (none) -> the-card:SO-8_L4.9-W3.9-P1.27-LS6.0-BL
- U3: footprint (none) -> the-card:LGA-14_L3.0-W2.5-P0.50-TL
- U4: footprint (none) -> the-card:DFN-4_L1.5-W1.5-P0.80-TL-EP
- U5: footprint (none) -> the-card:TDFN-8_L2.0-W2.0-P0.50-BL-EP1.2
- U6: footprint (none) -> the-card:ESOP-8_L4.9-W3.9-P1.27-LS6.0-BL-EP
- U7: footprint (none) -> the-card:SOT-23-6_L2.9-W1.6-P0.95-LS2.8-BR
- U8: footprint (none) -> the-card:TSSOP-8_L4.4-W3.0-P0.65-LS6.4-BL-2
- U9: footprint (none) -> the-card:SOT-23-5_L3.0-W1.7-P0.95-LS2.8-BL
Connections:
- net BAT_NEG is gone; now on an unnamed net: C_dprot.2, U7.1 (DOUT), U7.6 (VSS), U8.2 (S1), U8.3 (S1), U8.5 (G2)
- net N$10 is gone; now on an unnamed net: C_dprot.1, R_dvcc.2, U7.5 (VDD)
- net N$7 is gone; now on an unnamed net: J1.A6 (DP1), J1.B6 (DP2), U10.3
- net EPD_DC: no longer J2.1, J2.10, J2.12, J2.13, J2.14, J2.2, J2.3, J2.4, J2.5, J2.6, J2.7, J2.9, U1.15 (IO3), U1.17 (IO9), U1.18 (IO10), U1.19 (IO11), U1.20 (IO12), U1.22 (IO14), U2.7 (GPO)
- net ~CHRG: now also R_chrg.2, U6.7 (~{CHRG})
- net at R_prog.1, U6.2 (PROG): no longer R_chrg.2, U6.7 (~{CHRG})
- net FET_DRAIN: now reaches U8.1 (D12), U8.8 (D12)
- net LED_DIN: now reaches D1.4 (DIN), U1.25 (IO48)
- net N$1: no longer names the net of C_en.1, R_en.2, U1.3 (EN)
- net N$11: no longer names the net of R_dvm.2, U7.2 (VM)
- net N$3: no longer names the net of C_vb.1, R_vbh.2, R_vbl.1, U1.39 (IO1)
- net N$4: no longer names the net of J1.A5 (CC1), R_cc1.1
- net N$5: no longer names the net of J1.B5 (CC2), R_cc2.1
- net N$6: no longer names the net of J1.A7 (DN1), J1.B7 (DN2), U10.1
- new net EPD_BUSY: J2.9, U1.19 (IO11)
- new net EPD_CS: J2.12, U1.20 (IO12)
- new net EPD_GDR: J2.2
- new net EPD_NC1: J2.1
- new net EPD_NC4: J2.4
- new net EPD_RESE: J2.3
- new net EPD_RST: J2.10, U1.22 (IO14)
- new net EPD_SCLK: J2.13, U1.18 (IO10)
- new net EPD_SDA: J2.14, U1.17 (IO9)
- new net EPD_TSCL: J2.6
- new net EPD_TSDA: J2.7
- new net EPD_VSH2: J2.5
- new net NFC_IRQ: U1.15 (IO3), U2.7 (GPO)
Other:
- note added: "3.3 V regulation and fuel gauge"
- note added: "Cell protection"
- note added: "Controller, boot straps, decoupling, and battery ADC"
- note added: "GDEY029T94 24-pin FPC interface"
- note added: "I2C pull-ups"
- note added: "Motion and environmental sensors"
- note added: "NFC dynamic tag"
- note added: "Named labels keep long inter-block connections readable."
- note added: "Panel booster and high-voltage pins remain named for PCB review."
- note added: "Status LED"
- note added: "Switched peripheral rails"
- note added: "USB-C input, ESD, and charger"
- note added: "User buttons with hardware debounce"
- company: ESP32-S3 e-paper smart badge -> the-card
- title: the-card -> the-card - ESP32-S3 e-paper smart badge
