File: hardware/the-card.kicad_pcb (KiCad board)
At the start: 4 copper layers, 54 x 85.6 mm, 75 parts, among them J1 TYPE-C-31-M-12, J2 FH12-24S-0.5SH(55), J3 S2B-PH-SM4-TB(LF)(SN), Q1 SI2301CDS-T1-GE3, Q2 SI2301CDS-T1-GE3, Q3 SI1308EDL-T1-GE3, SW1 TS-1187A-B-A-B, SW2 TS-1187A-B-A-B, SW3 TS-1187A-B-A-B, SW4 TS-1187A-B-A-B, U1 ESP32-S3-WROOM-1-N16R8, U10 USBLC6-2SC6, U2 ST25DV04KC-IE8S3, U3 LSM6DSOTR, U4 SHT40-BD1B-R2, U5 MAX17048G+T10, U6 TP4056_C382139, U7 DW01A_C18164398, U8 8205A, U9 ME6211C33M5G-N

Commit message: fix(hardware): restore schematic PCB parity
Connections:
- net Net-(D2-K) renamed EPD_PUMP
- net Net-(D4-A) renamed EPD_SW
- net Net-(J3-Pin_2) renamed BAT_NEG
